File: BLDCdrv/BLDCdrv.kicad_pcb (KiCad board)
At the start: 2 copper layers, 110 x 60 mm, 29 parts, among them IC1 DRV8300DIPWR, J1 Screw_Terminal_01x02, J2 Conn_01x08_Male, J3 Screw_Terminal_01x03, Q1 IRF540N, Q2 IRF540N, Q3 IRF540N, Q4 IRF540N, Q5 IRF540N, Q6 IRF540N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

Commit message: Update wire width, mount holes and silkprint info
Parts:
- added REF**: MountingHole_3.2mm_M3, MountingHole:MountingHole_3.2mm_M3, F.Cu at (90.1, 122.2)
- added REF**: MountingHole_3.2mm_M3, MountingHole:MountingHole_3.2mm_M3, F.Cu at (90.1, 69.2)
- added REF**: MountingHole_3.2mm_M3, MountingHole:MountingHole_3.2mm_M3, F.Cu at (193.1, 122.2)
- added REF**: MountingHole_3.2mm_M3, MountingHole:MountingHole_3.2mm_M3, F.Cu at (193.1, 69.2)
- moved G*** 71.2 mm to (165.8, 113.6)
- moved U1 8.63 mm to (94.4, 108.6), turned to 90 degrees
Routing:
- net GNDREF: track 183.6 -> 193.7 mm
- net +BATT: track 133.2 -> 125.7 mm
- net Net-(JP1-Pad1): track 15.8 -> 12.5 mm
- net Net-(IC1-Pad13): track 76.4 -> 78.7 mm
- net Net-(IC1-Pad16): track 53.8 -> 54.7 mm
- net Net-(C6-Pad1): track 22.4 -> 23.2 mm
- net Net-(C5-Pad2): track 168.3 -> 167.6 mm
- net Net-(C7-Pad2): track 127.8 -> 128.5 mm
- net Net-(C5-Pad1): track 27.6 -> 28.2 mm
- net Net-(IC1-Pad6): track 21.1 -> 21.7 mm
Other:
- board text added: "+5V"
- board text added: "+Source Input"
- board text added: "3-phase BLDC Motor Drive"
- board text added: "GND"
- board text added: "ICT 2024"
- board text added: "Inverter output"
- board text added: "MCU Interface"
- board text added: "Phase A"
- board text added: "Phase B"
- board text added: "Phase C"

Commit message: Including gerberfiles for the first PCB prod.
Parts:
- moved G*** 1.99 mm to (166.4, 115.5)
