File: BLDCdrv/BLDCdrv.kicad_sch (KiCad schematic)
At the start: 28 parts, among them IC1 DRV8300DIPWR, J1 Screw_Terminal_01x02, J2 Conn_01x08_Male, J3 Screw_Terminal_01x03, Q1 IRF540N, Q2 IRF540N, Q3 IRF540N, Q4 IRF540N, Q5 IRF540N, Q6 IRF540N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

Commit message: Hasty checkin of current development projects...
Parts:
- R1, R2, R4, R5, R7, R8: value (none) -> 15; footprint (none) -> Resistor_THT:R_Axial_DIN0207_L6.3mm_D2.5mm_P10.16mm_Horizontal
- R3, R6, R9: value (none) -> 0; footprint (none) -> Resistor_THT:R_Axial_DIN0207_L6.3mm_D2.5mm_P10.16mm_Horizontal
