File: ELE302Lab/ELE302Lab.kicad_pcb (KiCad board)
At the start: 2 copper layers, 53.7 x 38.5 mm, 21 parts, among them J1 SSM-104-F-SH-TR, J2 SSM-103-L-SH-TR, J3 SSM-104-F-SH-TR, J4 USB_C_Receptacle_PowerOnly_6P, Q3 IMH3A, SW2 AYZ0202AGRLC, U1 LTC3525-5

Commit message: Last years (2024) ELE302 lab project.
Parts:
- removed J1: SSM-104-F-SH-TR, SSM_104_F_SH_TR:SAMTEC_SSM-104-F-SH-TR
- added C6: 47uF, Capacitor_SMD:C_1206_3216Metric_Pad1.33x1.80mm_HandSolder, F.Cu at (124.1, 73.2)
- added D2: CD4148W, Diode_SMD:D_0805_2012Metric, F.Cu at (130.1, 72.9)
- added J5: DB9_Female, Connector_Dsub:DSUB-9_Female_Horizontal_P2.77x2.84mm_EdgePinOffset9.90mm_Housed_MountingHolesOffset11.32mm, F.Cu at (116.4, 95.9)
- added Q1: FMB3946, Package_TO_SOT_SMD:TSOT-23-6_HandSoldering, F.Cu at (126.5, 78.3)
- added R10: 10k, Resistor_SMD:R_1206_3216Metric_Pad1.30x1.75mm_HandSolder, F.Cu at (146.7, 73.0)
- added R6: 10k, Resistor_SMD:R_1206_3216Metric_Pad1.30x1.75mm_HandSolder, F.Cu at (127.7, 88.8)
- added R7: 10k, Resistor_SMD:R_1206_3216Metric_Pad1.30x1.75mm_HandSolder, F.Cu at (129.2, 84.1)
- added R8: 10k, Resistor_SMD:R_1206_3216Metric_Pad1.30x1.75mm_HandSolder, F.Cu at (123.8, 84.1)
- added R9: 10k, Resistor_SMD:R_1206_3216Metric_Pad1.30x1.75mm_HandSolder, F.Cu at (152.6, 76.8)
- R1: value 5.1k -> 1k
- R3: value 1k -> 5.1k
- moved R4 10.6 mm to (161.7, 91.6), turned to 90 degrees
- moved R5 2.19 mm to (124.3, 94.8), turned to 90 degrees
- moved R1 0.32 mm to (170.6, 81.3), turned to 180 degrees
- moved BT1 0.10 mm to (123.5, 101.0)
Connections:
- Q3 pad 1: Net-(J1-03) -> Net-(Q3A-C1)
- R1 pad 1: Net-(J4-CC1) -> Net-(D1-A)
- R1 pad 2: Net-(J4-SHIELD) -> Net-(Q3A-C1)
- R2 pad 1: Net-(D1-A) -> Net-(J2-03)
- R2 pad 2: Net-(J1-03) -> Net-(D1-A)
- R3 pad 1: Net-(J2-03) -> Net-(J4-CC2)
- R3 pad 2: Net-(D1-A) -> Net-(J4-SHIELD)
- R4 pad 1: Net-(J4-CC2) -> Net-(J4-CC1)
Routing:
- net Net-(Q1B-C2): track 0.00 -> 49.3 mm, vias 0 -> 1
- net Net-(J1-03): track 45.5 -> 0.00 mm, vias 2 -> 0
- net Net-(D2-K): track 0.00 -> 43.6 mm
- net GNDREF: track 190.1 -> 217.0 mm, vias 8 -> 9
- net Net-(Q3A-C1): track 0.00 -> 26.5 mm, vias 0 -> 2
- net Net-(Q1B-B2): track 0.00 -> 21.2 mm, vias 0 -> 2
- net Net-(D2-A): track 0.00 -> 18.6 mm
- net Net-(J2-03): track 28.6 -> 38.0 mm
- net Net-(Q1A-B1): track 0.00 -> 8.13 mm
- net Net-(J4-CC2): track 15.1 -> 21.8 mm, vias 0 -> 2
- net Net-(D1-A): track 105.4 -> 111.9 mm, vias 4 -> 6
- net Net-(J4-CC1): track 10.8 -> 13.5 mm, vias 0 -> 2
- net Net-(D1-K): track 2.97 -> 5.69 mm
- net Net-(Q1A-C1): track 53.9 -> 51.4 mm, vias 2 -> 3
- net Net-(J4-SHIELD): track 79.3 -> 77.1 mm, vias 0 -> 2
Other:
- board size 53.7 x 38.5 mm -> 70.6 x 38.5 mm
