File: ELE302Lab/ELE302Lab.kicad_sch (KiCad schematic)
At the start: 20 parts, among them J1 SSM-104-F-SH-TR, J2 SSM-103-L-SH-TR, J3 SSM-104-F-SH-TR, J4 USB_C_Receptacle_PowerOnly_6P, Q3 IMH3A, SW2 AYZ0202AGRLC, U1 LTC3525-5

Commit message: Last years (2024) ELE302 lab project.
Parts:
- removed J1: SSM-104-F-SH-TR, SSM_104_F_SH_TR:SAMTEC_SSM-104-F-SH-TR, symbol SSM-104-F-SH-TR:SSM-104-F-SH-TR
- added C6: 47uF, Capacitor_SMD:C_1206_3216Metric_Pad1.33x1.80mm_HandSolder, symbol Device:C_Polarized
- added D2: CD4148W, Diode_SMD:D_0805_2012Metric, symbol Diode:CD4148W
- added J5: DB9_Female, Connector_Dsub:DSUB-9_Female_Horizontal_P2.77x2.84mm_EdgePinOffset9.90mm_Housed_MountingHolesOffset11.32mm, symbol Connector:DB9_Female
- added Q1: FMB3946, Package_TO_SOT_SMD:TSOT-23-6_HandSoldering, symbol Transistor_BJT:FMB3946
- added R10, R6, R7, R8, R9: 10k, Resistor_SMD:R_1206_3216Metric_Pad1.30x1.75mm_HandSolder, symbol Device:R
- renumbered R2 to R1, R3 to R2, R4 to R3, R1 to R4
Connections:
- net GNDREF: now also C6.2, J5.5, Q1.5 (E1), R7.1
- net at C3.1, C4.1, C5.1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: now also Q1.2 (E2), R9.2
- net at Q3.1 (C1), R1.2: now also R10.2
- net at Q3.2 (B2): now also Q1.6 (C1), R9.1
- new net: D2.1 (K), J5.3, R6.2
- new net: C6.1, D2.2 (A), R8.1
- new net: Q1.1 (B1), R6.1, R7.2
- new net: Q1.3 (B2), R10.1
- new net: J5.2, Q1.4 (C2), R8.2
Other:
- note added: "RF-RX"
- note added: "RF-TX"
- note added: "RS232-RX"
- note added: "RS232-TX"
- note added: "TTL-RX"
- note added: "TTL-TX"
- note removed: "From PC terminal"
- note removed: "Towards PC terminal"
- moved on the sheet: BT1, C1, C2, C3, C4, C5, D1, J2, J3, J4, L1, Q3A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
