File: BiathlonToyTarget/CorntrolHub/CorntrolHub.kicad_sch (KiCad schematic)
At the start: 32 parts, among them IC1 STM32G030K6T6, J1 Target1, J10 AudioJack3, J12 Barrel_Jack_Switch, J2 Target2, J3 Target3, J4 Target4, J5 Target5, J6 SWD, J7 DB9_Female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

Commit message: Checking in the current design and prod files.
Parts:
- J8: value Utility Pins -> Utility Pins
Other:
- note added: "7-seg HOURS (Blue-White)"
- note added: "7-seg Hundreth (Orange)"
- note added: "7-seg Minutes (Blue)"
- note added: "7-seg Seconds (Green-White)"
- note added: "CLOCK (Green)"
- note added: "STROBE (Brown-White)"
- note removed: "7-seg HOURS"
- note removed: "7-seg Hundreth"
- note removed: "7-seg Minutes"
- note removed: "7-seg Seconds"
- note removed: "CLOCK"
- note removed: "STROBE"
Changed lines of the file:
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@@
 (kicad_sch
-	(version 20231120)
+	(version 20250114)
 	(generator "eeschema")
-	(generator_version "8.0")
+	(generator_version "9.0")
 	(paper "A4")
+	(text "3V3"
+		(exclude_from_sim no)
+		(at 51.816 20.574 0)
+		(effects
+			(font
+				(size 1.27 1.27)
+			)
+		)
+	)
+	(text "7-seg HOURS (Blue-White)"
+		(exclude_from_sim no)
+		(at 140.716 175.514 0)
+		(effects
+			(font
+				(size 1.27 1.27)
+			)
+		)
+	)
+	(text "3V3"
+		(exclude_from_sim no)
+		(at 217.678 35.814 0)
+		(effects
+			(font
+				(size 1.27 1.27)
+			)
+		)
+	)
+	(text "ST-Link"
+		(exclude_from_sim no)
+		(at 208.28 21.59 0)
+		(effects
+			(font
+				(size 2 2)
+			)
+			(justify left bottom)
+		)
+	)
+	(text "Programming\nBoot loading sys mem"
+		(exclude_from_sim no)
+		(at 226.06 49.53 0)
+		(effects
+			(font
+				(size 2 2)
+			)
+			(justify left bottom)
+		)
+	)
+	(text "7-seg Hundreth (Orange)"
+		(exclude_from_sim no)
+		(at 139.7 183.388 0)
+		(effects
+			(font
+				(size 1.27 1.27)
+			)
+		)
+	)
+	(text "7-seg Seconds (Green-White)"
+		(exclude_from_sim no)
+		(at 141.986 180.848 0)
+		(effects
+			(font
+				(size 1.27 1.27)
+			)
+		)
+	)
+	(text "7-seg Minutes (Blue)"
+		(exclude_from_sim no)
+		(at 137.668 178.054 0)
+		(effects
+			(font
+				(size 1.27 1.27)
+			)
+		)
+	)
+	(text "CoverPWM"
+		(exclude_from_sim no)
+		(at 121.666 137.414 0)
+		(effects
+			(font
+				(size 1.27 1.27)
+			)
+		)
+	)
+	(text "TTL-RX"
+		(exclude_from_sim no)
+		(at 73.66 156.21 0)
+		(effects
+			(font
+				(size 1.778 1.5113)
+			)
+			(justify left bottom)
+		)
+	)
+	(text "RS232-RX"
+		(exclude_from_sim no)
+		(at 46.99 148.59 90)
+		(effects
+			(font
+				(size 2 2)
+			)
+			(justify right bottom)
+		)
+	)
+	(text "GND"
+		(exclude_from_sim no)
+		(at 217.424 30.734 0)
+		(effects
+			(font
+				(size 1.27 1.27)
+			)
+		)
+	)
+	(text "GND"
+		(exclude_from_sim no)
+		(at 33.528 41.148 0)
+		(effects
+			(font
+				(size 1.27 1.27)
+			)
+		)
+	)
+	(text "Hit-Intr"
+		(exclude_from_sim no)
+		(at 122.428 142.494 0)
+		(effects
+			(font
+				(size 1.27 1.27)
+			)
+		)
+	)
+	(text "STROBE (Brown-White)"
+		(exclude_from_sim no)
+		(at 139.446 170.434 0)
+		(effects
+			(font
+				(size 1.27 1.27)
+			)
+		)
+	)
+	(text "Start Stop-Watch"
+		(exclude_from_sim no)
+		(at 49.276 122.174 0)
+		(effects
+			(font
+				(size 1.27 1.27)
+			)
+		)
+	)
+	(text "CLOCK (Green)"
+		(exclude_from_sim no)
+		(at 135.382 172.974 0)
+		(effects
+			(font
+				(size 1.27 1.27)
+			)
+		)
+	)
+	(text "TTL-TX"
+		(exclude_from_sim no)
+		(at 86.36 135.89 0)
+		(effects
+			(font
+				(size 1.778 1.5113)
+			)
+			(justify left bottom)
+		)
+	)
+	(text "RS232-TX"
+		(exclude_from_sim no)
+		(at 41.91 148.59 90)
+		(effects
+			(font
+				(size 2 2)
+			)
+			(justify right bottom)
+		)
+	)
+	(text "battery and charging supply"
+		(exclude_from_sim no)
+		(at 239.268 151.638 0)
+		(effects
+			(font
+				(size 1.27 1.27)
+			)
+		)
+	)
+	(text "Manually reset targets"
+		(exclude_from_sim no)
+		(at 55.626 112.268 0)
+		(effects
+			(font
+				(size 1.27 1.27)
+			)
+		)
+	)
 	(junction
 		(at 140.97 114.3)
@@
 		)
 	)
-	(text "3V3"
-		(exclude_from_sim no)
-		(at 51.816 20.574 0)
-		(effects
-			(font
-				(size 1.27 1.27)
-			)
-		)
-	)
-	(text "7-seg HOURS "
-		(exclude_from_sim no)
-		(at 135.128 175.514 0)
-		(effects
-			(font
-				(size 1.27 1.27)
-			)
-		)
-	)
-	(text "3V3"
-		(exclude_from_sim no)
-		(at 217.678 35.814 0)
-		(effects
-			(font
-				(size 1.27 1.27)
-			)
-		)
-	)
-	(text "ST-Link"
-		(exclude_from_sim no)
-		(at 208.28 21.59 0)
-		(effects
-			(font
-				(size 2 2)
-			)
-			(justify left bottom)
-		)
-	)
-	(text "Programming\nBoot loading sys mem"
-		(exclude_from_sim no)
-		(at 226.06 49.53 0)
-		(effects
-			(font
-				(size 2 2)
-			)
-			(justify left bottom)
-		)
-	)
-	(text "7-seg Hundreth "
-		(exclude_from_sim no)
-		(at 136.144 183.134 0)
-		(effects
-			(font
-				(size 1.27 1.27)
-			)
-		)
-	)
-	(text "7-seg Seconds"
-		(exclude_from_sim no)
-		(at 135.128 180.594 0)
-		(effects
-			(font
-				(size 1.27 1.27)
-			)
-		)
-	)
-	(text "7-seg Minutes"
-		(exclude_from_sim no)
-		(at 134.874 178.054 0)
-		(effects
-			(font
-				(size 1.27 1.27)
-			)
-		)
-	)
-	(text "CoverPWM"
-		(exclude_from_sim no)
-		(at 121.666 137.414 0)
-		(effects
-			(font
-				(size 1.27 1.27)
-			)
-		)
-	)
-	(text "TTL-RX"
-		(exclude_from_sim no)
-		(at 73.66 156.21 0)
-		(effects
-			(font
-				(size 1.778 1.5113)
-			)
-			(justify left bottom)
-		)
-	)
-	(text "RS232-RX"
-		(exclude_from_sim no)
-		(at 46.99 148.59 90)
-		(effects
-			(font
-				(size 2 2)
-			)
-			(justify right bottom)
-		)
-	)
-	(text "GND"
-		(exclude_from_sim no)
-		(at 217.424 30.734 0)
-		(effects
-			(font
-				(size 1.27 1.27)
-			)
-		)
-	)
-	(text "GND"
-		(exclude_from_sim no)
-		(at 33.528 41.148 0)
-		(effects
-			(font
-				(size 1.27 1.27)
-			)
-		)
-	)
-	(text "Hit-Intr"
-		(exclude_from_sim no)
-		(at 122.428 142.494 0)
-		(effects
-			(font
-				(size 1.27 1.27)
-			)
-		)
-	)
-	(text "STROBE"
-		(exclude_from_sim no)
-		(at 132.08 170.434 0)
-		(effects
-			(font
-				(size 1.27 1.27)
-			)
-		)
-	)
-	(text "Start Stop-Watch"
-		(exclude_from_sim no)
-		(at 49.276 122.174 0)
-		(effects
-			(font
-				(size 1.27 1.27)
-			)
-		)
-	)
-	(text "CLOCK"
-		(exclude_from_sim no)
-		(at 131.572 172.974 0)
-		(effects
-			(font
-				(size 1.27 1.27)
-			)
-		)
-	)
-	(text "TTL-TX"
-		(exclude_from_sim no)
-		(at 86.36 135.89 0)
-		(effects
-			(font
-				(size 1.778 1.5113)
-			)
-			(justify left bottom)
-		)
-	)
-	(text "RS232-TX"
-		(exclude_from_sim no)
-		(at 41.91 148.59 90)
-		(effects
-			(font
-				(size 2 2)
-			)
-			(justify right bottom)
-		)
-	)
-	(text "battery and charging supply"
-		(exclude_from_sim no)
-		(at 239.268 151.638 0)
-		(effects
-			(font
-				(size 1.27 1.27)
-			)
-		)
-	)
-	(text "Manually reset targets"
-		(exclude_from_sim no)
-		(at 55.626 112.268 0)
-		(effects
-			(font
-				(size 1.27 1.27)
-			)
-		)
-	)
 	(global_label "Servo2pwm"
 		(shape input)
@@
 			)
 		)
-		(property "Value" "Utility Pins "
+		(property "Value" "Utility Pins"
 			(at 39.37 17.78 0)
 			(effects
@@
 		)
 	)
+	(embedded_fonts no)
 )
