File: BiathlonToyTarget/SignalsPort/SignalsPort.kicad_pcb (KiCad board)
At the start: 2 copper layers, 38 x 29.7 mm, 5 parts, among them J1 Servo, J2 HitSens, J3 SignalsPort

Commit message: Checking in the current design and prod files.
Parts:
- removed REF** (x2): MountingHole_3.2mm_M3, MountingHole:MountingHole_3.2mm_M3
- added C1: 100µF 16V, Capacitor_SMD:C_Elec_6.3x7.7, F.Cu at (128.9, 109.1)
- added D1: LED, LED_SMD:LED_0805_2012Metric_Pad1.15x1.40mm_HandSolder, F.Cu at (131.9, 96.5)
- added H1: MountingHole, MountingHole:MountingHole_3.2mm_M3, F.Cu at (150.6, 89.7)
- added H2: MountingHole, MountingHole:MountingHole_3.2mm_M3, F.Cu at (119.6, 112.6)
- added R1: 1k, Resistor_SMD:R_0805_2012Metric_Pad1.20x1.40mm_HandSolder, F.Cu at (128.2, 94.9)
- added R2: 1k, Resistor_SMD:R_0805_2012Metric_Pad1.20x1.40mm_HandSolder, F.Cu at (141.2, 103.1)
- added U1: CPC1017N, Package_SO:SOP-4_3.8x4.1mm_P2.54mm, F.Cu at (135.7, 101.5)
Connections:
- J3 pad 1: Net-(J2-Pin_3) -> Net-(D1-A)
- J3 pad 3: Net-(J1-Pin_3) -> Net-(J3-Pin_3)
- J3 pad MP: GNDREF -> (no net)
Routing:
- net Net-(D1-A): track 0.00 -> 37.0 mm
- net GNDREF: track 92.9 -> 120.7 mm
- net Net-(J2-Pin_3): track 29.7 -> 2.88 mm
- net Net-(J3-Pin_3): track 0.00 -> 13.3 mm
- net Net-(J1-Pin_3): track 31.3 -> 19.6 mm
- net +6V: track 64.9 -> 69.6 mm
- net Net-(R2-Pad2): track 0.00 -> 4.19 mm
