File: BiathlonToyTarget/SignalsPort/SignalsPort.kicad_sch (KiCad schematic)
At the start: 3 parts, among them J1 Servo, J2 HitSens, J3 SignalsPort

Commit message: Checking in the current design and prod files.
Parts:
- added C1: 100µF 16V, Capacitor_SMD:C_Elec_6.3x7.7, symbol Device:C_Polarized
- added D1: LED, LED_SMD:LED_0805_2012Metric_Pad1.15x1.40mm_HandSolder, symbol Device:LED
- added H1, H2: MountingHole, MountingHole:MountingHole_3.2mm_M3, symbol Mechanical:MountingHole
- added R1, R2: 1k, Resistor_SMD:R_0805_2012Metric_Pad1.20x1.40mm_HandSolder, symbol Device:R
- added U1: CPC1017N, Package_SO:SOP-4_3.8x4.1mm_P2.54mm, symbol Relay_SolidState:CPC1017N
Connections:
- net +6V: now also C1.1, U1.4
- net GNDREF: now also C1.2, D1.1 (K), R2.1
- net at J3.1 (Pin_1): now also D1.2 (A), R1.1; no longer J2.3 (Pin_3)
- net at J3.3 (Pin_3): now also U1.1; no longer J1.3 (Pin_3)
- new net: R2.2, U1.2
- new net: J2.3 (Pin_3), R1.2
- new net: J1.3 (Pin_3), U1.3
Other:
- moved on the sheet: J1, J2, J3
