File: BiathlonToyTarget/TargetHitDetector/TargetHitDetector.kicad_sch (KiCad schematic)
At the start: 14 parts, among them J1 Screw_Terminal_01x03, U1 LM321, U2 LM321

Commit message: Checking in the current design and prod files.
Parts:
- added H1, H2, H3, H4: MountingHole, MountingHole:MountingHole_3.2mm_M3, symbol Mechanical:MountingHole
- added R4: 1k, Resistor_SMD:R_1206_3216Metric_Pad1.30x1.75mm_HandSolder, symbol Device:R
- C2: value 0.47u -> 1µF
Connections:
- net Earth: now also R4.1
- net at C2.1, D4.1 (K), R3.2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: now also R4.2
