File: Big7segDisplayDrv/Big7segDisplayDrv.kicad_pcb (KiCad board)
At the start: 2 copper layers, 27 parts, among them J1 Screw_Terminal_01x02, J10 Barrel_Jack_Switch, J2 Screw_Terminal_01x02, J3 Screw_Terminal_01x03, J4 DB9_Male_MountingHoles, J5 DB9_Male_MountingHoles, J6 DB9_Male_MountingHoles, J7 DB9_Male_MountingHoles, Q1 BC548, Q2 BC548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

Commit message: First version for PCB production.
Parts:
- added G***: LOGO, uia-logo:uiaLogo, F.Cu at (154.9, 96.4)
- added REF**: MountingHole_3.2mm_M3, MountingHole:MountingHole_3.2mm_M3, F.Cu at (100.9, 68.8)
- added REF**: MountingHole_3.2mm_M3, MountingHole:MountingHole_3.2mm_M3, F.Cu at (100.8, 131.8)
- added REF**: MountingHole_3.2mm_M3, MountingHole:MountingHole_3.2mm_M3, F.Cu at (169.9, 68.8)
- added REF**: MountingHole_3.2mm_M3, MountingHole:MountingHole_3.2mm_M3, F.Cu at (169.9, 131.8)
- Q1, Q2, Q3, Q4, Q5, Q6: footprint Package_TO_SOT_THT:TO-92_Inline -> Package_TO_SOT_THT:TO-92_HandSolder
- moved J10 6.72 mm to (159.6, 100.8)
- moved J1 6.50 mm to (101.3, 85.0)
- moved J2 6.50 mm to (101.3, 95.7)
- moved J3 6.50 mm to (101.3, 106.4)
- moved Q3 1.36 mm to (130.6, 96.2)
- moved Q4 1.36 mm to (130.6, 102.5)
- moved Q5 1.36 mm to (130.6, 108.8)
- moved Q6 1.36 mm to (130.6, 115.1)
- moved Q1 1.36 mm to (130.6, 83.7)
- moved Q2 1.36 mm to (130.6, 90.0)
Routing:
- net VCC: track 165.0 -> 194.8 mm
- net /serData2: track 1.65 -> 14.4 mm
- net /serData1: track 7.52 -> 14.0 mm
- net /serData4: track 8.71 -> 15.2 mm
- net /serData3: track 8.22 -> 14.7 mm
- net /Strobe: track 9.46 -> 16.0 mm
- net /Clk: track 8.96 -> 15.5 mm
- net /ssd1: track 85.0 -> 89.8 mm
- net /sStrobe: track 172.4 -> 175.7 mm
- net GNDREF: track 206.2 -> 208.9 mm, vias 0 -> 2
- net /ssd2: track 51.4 -> 53.3 mm
- net /sClk: track 123.2 -> 125.1 mm
- net /ssd3: track 54.5 -> 56.2 mm
- net /ssd4: track 37.5 -> 38.9 mm
Other:
- board outline added: 76 x 70 mm

Commit message: Checking in current design and production files.
Parts:
- removed J1, J2: Screw_Terminal_01x02, TerminalBlock:TerminalBlock_bornier-2_P5.08mm
- removed J3: Screw_Terminal_01x03, TerminalBlock:TerminalBlock_bornier-3_P5.08mm
- removed REF** (x4): MountingHole_3.2mm_M3, MountingHole:MountingHole_3.2mm_M3
- added G***: LOGO, uia-logo:uiaLogo, F.Cu at (98.2, 76.8)
- added J8: 8P8C, Connector_RJ:RJ45_Amphenol_54602-x08_Horizontal, F.Cu at (107.2, 94.9)
- moved G*** 62.2 mm to (98.6, 122.9)
Connections:
- J4 pad 0: Net-(J4-Pad0) -> GNDREF
- J5 pad 0: Net-(J4-Pad0) -> GNDREF
- J6 pad 0: Net-(J4-Pad0) -> GNDREF
- J7 pad 0: Net-(J4-Pad0) -> GNDREF
Routing:
- net GNDREF: track 208.9 -> 227.4 mm
- net /serData3: track 14.7 -> 6.12 mm
- net /serData4: track 15.2 -> 11.1 mm
- net /serData1: track 14.0 -> 17.1 mm
- net /Clk: track 15.5 -> 12.8 mm
- net /Strobe: track 16.0 -> 17.1 mm
Other:
- board size 76 x 70 mm -> 80.7 x 70 mm
