File: Big7segDisplayDrv/Big7segDisplayDrv.kicad_sch (KiCad schematic)
At the start: 27 parts, among them J1 Screw_Terminal_01x02, J10 Barrel_Jack_Switch, J2 Screw_Terminal_01x02, J3 Screw_Terminal_01x03, J4 DB9_Male_MountingHoles, J5 DB9_Male_MountingHoles, J6 DB9_Male_MountingHoles, J7 DB9_Male_MountingHoles, Q1 BC548, Q2 BC548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

Commit message: Checking in current design and production files.
Parts:
- removed J1, J2: Screw_Terminal_01x02, TerminalBlock:TerminalBlock_bornier-2_P5.08mm, symbol Connector:Screw_Terminal_01x02
- removed J3: Screw_Terminal_01x03, TerminalBlock:TerminalBlock_bornier-3_P5.08mm, symbol Connector:Screw_Terminal_01x03
- added J8: 8P8C, Connector_RJ:RJ45_Amphenol_54602-x08_Horizontal, symbol Connector:8P8C
Connections:
- net Clk: now also J8.6
- net GNDREF: now also J4.0 (PAD), J5.0 (PAD), J6.0 (PAD), J7.0 (PAD), J8.1, J8.8
- net Strobe: now also J8.7
- net serData1: now also J8.2
- net serData2: now also J8.3
- net serData3: now also J8.4
- net serData4: now also J8.5
Other:
- moved on the sheet: R10, R11, R12, R7, R8, R9
