File: BLDCsensDrv/BLDCsensDrv.kicad_pcb (KiCad board)
At the start: 2 copper layers, 106 x 65 mm, 72 parts, among them J1 Screw_Terminal_01x02, J20 Utility Pins, J21 UART PORT#1, J22 UART PORT#2, J23 DB9_Female, J24 DB9_Female, J25 SWD, J4 Ctrl-Port, J5 Monitor, J6 Screw_Terminal_01x03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

Commit message: Hasty checkin of current development projects...
Parts:
- removed REF** (x4): MountingHole_3.2mm_M3, MountingHole:MountingHole_3.2mm_M3
Connections:
- net Net-(J1-Pin_1) renamed PVDD
